File: kicad/v5/v5.sch (KiCad schematic (older format))
At the start: 44 parts, among them J1 BNC, J1-1 Head1_1, J1-2 Head1_1, J2 BNC, J2-1 Head1_1, J2-2 Head1_1, J2-3 Head1_1, J3 Green, J3-1 Head1_1, J3-2 Head1_1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

Commit message: Schematic:  v5b - Floating transformer output.  Output connector shield     is grounded on pin 4.
Connections:
- net OGnd renamed Shield
- net Shield: no longer J7.1b (Pin_1b), J7.4b (Pin_4b)
- no-connect marks 0 -> 2
Other:
- note added: "Ground Connection"
- note removed: "Optional Ground Connection"
Changed lines of the file:
@@
 encoding utf-8
 Sheet 1 1
-Title "Piezo AC Driver - v5, Protoboard"
-Date "2019-04-08"
+Title "Piezo AC Driver - v5b, Protoboard"
+Date "2019-05-15"
 Rev ""
 Comp "William A. Hudson"
 Comment1 "https://github.com/wahudson/piezo_ac_drive"
-Comment2 ""
-Comment3 ""
+Comment2 "v5  - Power reverse polarity protection."
+Comment3 "v5b - Floating transformer output.  Output shield grounded."
 Comment4 ""
 $EndDescr
@@
 $EndComp
 Wire Wire Line
-	6800 5500 6900 5500
-Wire Wire Line
-	6900 5500 6900 4800
-Wire Wire Line
-	6900 4800 7500 4800
+	7200 4800 7500 4800
 Wire Wire Line
 	6800 5600 7000 5600
@@
 Wire Wire Line
 	7100 5200 7500 5200
-Wire Wire Line
-	6800 5800 8400 5800
 Wire Wire Line
 	8400 5800 8400 5200
@@
 Wire Wire Line
 	6200 6000 6300 6000
-Wire Wire Line
-	6800 5800 6850 5750
-Wire Wire Line
-	6850 5750 6850 5550
-Wire Wire Line
-	6850 5550 6800 5500
-Connection ~ 6800 5800
-Connection ~ 6800 5500
 Text Label 7200 4800 0    50   ~ 0
-OGnd
+Shield
 Text Label 7200 5000 0    50   ~ 0
 X_Vsp
@@
 X_Vsn
 Text Label 8250 5200 0    50   ~ 0
-OGnd
+Shield
 Text Label 8250 5000 0    50   ~ 0
 Y_Vsp
@@
 Text Notes 5650 2400 0    50   ~ 0
 100V
-Wire Wire Line
-	6800 5800 6850 5850
 Wire Wire Line
 	1600 5550 1750 5600
@@
 Text Notes 7450 4400 0    50   ~ 0
 High Voltage Output
-Text Notes 1550 4400 0    100  ~ 0
+Text Notes 1700 4600 0    100  ~ 0
 2-Channel Prototype
-Text Notes 450  5300 0    50   ~ 0
+Text Notes 600  5300 0    50   ~ 0
 Power  V= 9 to 24 Vdc
 Text Notes 5650 5050 0    50   ~ 0
@@
 	6000 3000 6100 3000
 Text Notes 3700 7300 0    50   ~ 0
-Optional Ground Connection
+Ground Connection
 $Comp
 L Diode:1N4002 D11
@@
 Reverse Polarity Protection
 Wire Wire Line
-	6850 5850 6300 7200
-Wire Wire Line
-	1750 7200 6300 7200
+	1750 7200 5700 7200
 Wire Notes Line
 	3350 5100 3350 7100
@@
 Text Notes 1650 900  0    100  ~ 0
 AC_Driver_Stepup
+Wire Wire Line
+	8400 5800 7200 5800
+Wire Wire Line
+	7200 5800 5700 7200
+NoConn ~ 6800 5500
+NoConn ~ 6800 5800
 $EndSCHEMATC
